File: Motor Driver Board/Motor Driver MK1.brd (EAGLE design)
At the start: 100 x 81.3 mm, 98 parts, among them IC1 REG1117

Commit message: Finished up control board. Pending second review.
Parts:
- removed AC3: (no value), rcl:C0805
- moved LED2 0.32 mm to (76.2, 65.7)
- moved RLED1 0.32 mm to (80.0, 65.7)
- flipped AC1 to the top, turned to 0 degrees
- turned AHOME_UP to 180 degrees
- turned EN_IN to 0 degrees
- turned FAULT_IN to 0 degrees
- flipped XC1 to the top, turned to 0 degrees
- flipped YC1 to the top, turned to 0 degrees
- flipped ZC1 to the top, turned to 0 degrees
- turned ZHOME_UP to 180 degrees
Connections:
- net XHOME_UP renamed N$64
- net GND: no longer AC3.2
- net VCC: no longer AC3.1
Routing:
- net GND: track 710.2 -> 771.4 mm
- net VCC: track 280.0 -> 313.1 mm
- net N$89: track 0.00 -> 13.2 mm, vias 0 -> 2
- net N$48: track 0.00 -> 13.2 mm, vias 0 -> 2
- net N$87: track 3.96 -> 12.6 mm, vias 0 -> 2
- net N$75: track 0.00 -> 7.25 mm
- net N$73: track 0.00 -> 5.61 mm
- net N$69: track 0.00 -> 4.34 mm
- net N$67: track 4.34 -> 0.00 mm
- net N$64: track 17.8 -> 13.5 mm, vias 0 -> 2
- net N$68: track 0.00 -> 3.07 mm
- net N$65: track 0.00 -> 3.07 mm
- net N$56: track 179.8 -> 182.8 mm
- net N$92: track 8.26 -> 10.8 mm
- net N$77: track 25.3 -> 27.8 mm
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Other:
- board size 100 x 81.3 mm -> 83.5 x 69.2 mm
- board text added: "2013"
- board text added: "EVAN MILTON"
- board text added: "Use Pololu DRV8825 or A4988"

Commit message: 8+ hours since last remote commit. Going to let it sit for now.
Parts:
- removed U$1: RASPBERRY-PI, RaspberryPi:RASPBERRY-PI
Routing:
- net VCC: track 313.1 -> 310.0 mm
Other:
- board size 83.5 x 69.2 mm -> 85.1 x 69.2 mm

Commit message: added comments, more cleanup.
Signed-off-by: Evan Milton <evan@bp2e.net>
Parts:
- AC1, XC1, YC1, ZC1: value (none) -> 100uF
- AC2, AC3, XC2, XC3, YC2, YC3, ZC2, ZC3: value (none) -> 100nF
- AHOME_OUT, FAULT_OUT, XHOME_OUT, YHOME_OUT, ZHOME_OUT: value 100 -> 1k
- AHOME_UP, FAULT_UP, XHOME_UP, YHOME_UP, ZHOME_UP: value 1k -> 100k
- EN_IN: value (none) -> 330
- renumbered AC4 to XC3, AC5 to YC3, AC6 to ZC3, AC7 to AC3
